File: hardware/EMS_BUS.kicad_sch (KiCad schematic)
At the start: 49 parts, among them IC1 LM393D, IC2 LT1129CST5, J1 SML, J2 PWR, J3 1Wire, Q2 BSS123, U1 ESP32-WROOM-32D

Commit message: Dokumentation erstellt
Parts:
- added D4, D5: LED, LED_THT:LED_D3.0mm_Clear, symbol Device:LED
Connections:
- net GND: now also D4.1 (K), D5.1 (K)
- net at R7.2, USER1.2 (A): now also D5.2 (A)
- net at PWR1.2 (A), R2.2: now also D4.2 (A)
Other:
- moved on the sheet: H1, H2, H3, H4
