File: hardware/EMS_BUS.kicad_pcb (KiCad board)
At the start: 2 copper layers, 74.9 x 59.7 mm, 49 parts, among them IC1 LM393D, IC2 LT1129CST5, J1 SML, J2 PWR, J3 1Wire, Q2 BSS123, U1 ESP32-WROOM-32D

Commit message: Dokumentation erstellt
Parts:
- added D4: LED, LED_THT:LED_D3.0mm_Clear, F.Cu at (153.9, 116.8)
- added D5: LED, LED_THT:LED_D3.0mm_Clear, F.Cu at (153.9, 110.6)
- moved R17 0.25 mm to (136.3, 96.4)
- moved R16 0.13 mm to (138.1, 96.5)
Routing:
- net Net-(PWR1-Pad2): track 1.69 -> 4.18 mm
- net Net-(R7-Pad2): track 1.69 -> 4.08 mm

Commit message: kleine Änderungen add gerber.zip
Parts:
- J3: footprint Connector_JST:JST_XA_B03B-XASK-1-A_1x03_P2.50mm_Vertical -> Connector_JST:JST_XA_B03B-XASK-1_1x03_P2.50mm_Vertical
Routing:
- net Net-(D3-Pad2): track 12.5 -> 11.4 mm
